Commit message: progs: added roobot wheels to urdf file

File: src/udacity_bot/urdf/udacity_bot.xacro (robot description, xacro)
@@ -78,7 +78,88 @@
       </geometry>
     </visual>
-    <!-- -->
-    <!-- -->
-    <!-- -->
   </link>
+  <!-- left_wheel -->
+  <link name="left_wheel">
+   <collision name='left_wheel_collision'>
+      <origin xyz="0 0 0" rpy=" 0 1.5707 1.5707"/>
+      <geometry>
+        <cylinder radius="0.1" length="0.05"/>
+      </geometry>
+      <surface>
+        <friction>
+          <ode>
+            <mu>0</mu>
+            <mu2>0</mu2>
+            <slip1>1.0</slip1>
+            <slip2>1.0</slip2>
+          </ode>
+        </friction>
+      </surface>
+    </collision>
+    <inertial>
+      <mass value="5.0"/>
+      <origin xyz="0.0 0 0" rpy=" 0 1.5707 1.5707"/>
+      <inertia
+          ixx="0.1" ixy="0" ixz="0"
+          iyy="0.1" iyz="0"
+          izz="0.1"
+      />
+    </inertial>
+    <visual name='left_wheel_visual'>
+      <origin xyz="0 0 0" rpy=" 0 1.5707 1.5707"/>
+      <geometry>
+        <cylinder radius="0.1" length="0.05"/>
+      </geometry>
+    </visual>
+  </link>
+  <joint type="continuous" name="left_wheel_hinge">
+      <origin xyz="0 0.15 0" rpy="0 0 0"/>
+      <child link="left_wheel"/>
+      <parent link="chassis"/>
+      <axis xyz="0 1 0" rpy="0 0 0"/>
+      <limit effort="10000" velocity="1000"/>
+      <joint_properties damping="1.0" friction="1.0"/>
+  </joint>
+  <!-- right_wheel -->
+ <link name="right_wheel">
+   <collision name='right_wheel_collision'>
+      <origin xyz="0 0 0" rpy=" 0 1.5707 1.5707"/>
+      <geometry>
+        <cylinder radius="0.1" length="0.05"/>
+      </geometry>
+      <surface>
+        <friction>
+          <ode>
+            <mu>0</mu>
+            <mu2>0</mu2>
+            <slip1>1.0</slip1>
+            <slip2>1.0</slip2>
+          </ode>
+        </friction>
+      </surface>
+    </collision>
+    <inertial>
+      <mass value="5.0"/>
+      <origin xyz="0.0 0 0" rpy=" 0 1.5707 1.5707"/>
+      <inertia
+          ixx="0.1" ixy="0" ixz="0"
+          iyy="0.1" iyz="0"
+          izz="0.1"
+      />
+    </inertial>
+    <visual name='right_wheel_visual'>
+      <origin xyz="0 0 0" rpy=" 0 1.5707 1.5707"/>
+      <geometry>
+        <cylinder radius="0.1" length="0.05"/>
+      </geometry>
+    </visual>
+  </link>
+  <joint type="continuous" name="right_wheel_hinge">
+      <origin xyz="0 -0.15 0" rpy="0 0 0"/>
+      <child link="right_wheel"/>
+      <parent link="chassis"/>
+      <axis xyz="0 1 0" rpy="0 0 0"/>
+      <limit effort="10000" velocity="1000"/>
+      <joint_properties damping="1.0" friction="1.0"/>
+  </joint>
 </robot>

Commit message: progs: added laser range finder

File: src/udacity_bot/urdf/udacity_bot.xacro (robot description, xacro)
@@ -123,5 +123,5 @@
   </joint>
   <!-- right_wheel -->
- <link name="right_wheel">
+  <link name="right_wheel">
    <collision name='right_wheel_collision'>
       <origin xyz="0 0 0" rpy=" 0 1.5707 1.5707"/>
@@ -164,3 +164,63 @@
       <joint_properties damping="1.0" friction="1.0"/>
   </joint>
+  <!-- camera -->
+  <link name="camera">
+   <collision name='camera_collision'>
+      <origin xyz="0 0 0" rpy=" 0 0 0"/>
+      <geometry>
+        <box size="0.05"/>
+      </geometry>
+    </collision>
+    <inertial>
+      <mass value="0.1"/>
+      <origin xyz="0 0 0" rpy=" 0 0 0"/>
+      <inertia
+          ixx="1e-6" ixy="0" ixz="0"
+          iyy="1e-6" iyz="0"
+          izz="1e-6"
+      />
+    </inertial>
+    <visual name='camera_visual'>
+      <origin xyz="0 0 0" rpy=" 0 0 0"/>
+      <geometry>
+        <box size="0.05"/>
+      </geometry>
+    </visual>
+  </link>
+  <joint type="fixed" name="camera_joint">
+      <origin xyz="0.2 0 0" rpy="0 0 0"/>
+      <child link="camera"/>
+      <parent link="chassis"/>
+      <axis xyz="1 0 0" rpy="0 0 0"/>
+  </joint>
+  <!-- hokuyo laser range finder -->
+  <link name="hokuyo">
+   <collision name='hokuyo_collision'>
+      <origin xyz="0 0 0" rpy=" 0 0 0"/>
+      <geometry>
+        <box size="0.1"/>
+      </geometry>
+    </collision>
+    <inertial>
+      <mass value="0.1"/>
+      <origin xyz="0 0 0" rpy=" 0 0 0"/>
+      <inertia
+          ixx="1e-6" ixy="0" ixz="0"
+          iyy="1e-6" iyz="0"
+          izz="1e-6"
+      />
+    </inertial>
+    <visual name='hokuyo_visual'>
+      <origin xyz="0 0 0" rpy=" 0 0 0"/>
+      <geometry>
+        <mesh filename="package://udacity_bot/meshes/hokuyo.dae"/>
+      </geometry>
+    </visual>
+  </link>
+  <joint type="fixed" name="hokuyo_joint">
+      <origin xyz="0.15 0 0.1" rpy="0 0 0"/>
+      <child link="hokuyo"/>
+      <parent link="chassis"/>
+      <axis xyz="1 0 0" rpy="0 0 0"/>
+  </joint>
 </robot>

Commit message: docs: added robot_4

File: src/udacity_bot/urdf/udacity_bot.xacro (robot description, xacro)
@@ -184,5 +184,5 @@
       <origin xyz="0 0 0" rpy=" 0 0 0"/>
       <geometry>
-        <box size="0.05"/>
+        <box size="0.05 0.05 0.05"/>
       </geometry>
     </visual>
@@ -196,8 +196,8 @@
   <!-- hokuyo laser range finder -->
   <link name="hokuyo">
-   <collision name='hokuyo_collision'>
-      <origin xyz="0 0 0" rpy=" 0 0 0"/>
-      <geometry>
-        <box size="0.1"/>
+    <collision name='hokuyo_collision'>
+      <origin xyz="0 0 0" rpy=" 0 0 0"/>
+      <geometry>
+        <box size="0.1 0.1 0.1"/>
       </geometry>
     </collision>

Commit message: progs: added gazebo plugin and materials

File: src/udacity_bot/urdf/udacity_bot.xacro (robot description, xacro)
@@ -2,4 +2,6 @@
 <!-- Udacity Robot -->
 <robot name="udacity_bot" xmlns:xacro="http://www.ros.org/wiki/xacro">
+  <!-- material properties -->
+  <xacro:include filename="$(find udacity_bot)/urdf/common_properties.xacro"/>
   <!-- robot_footprint -->
   <link name="robot_footprint"></link>
@@ -32,4 +34,5 @@
         <box size=".4 .2 .1"/>
       </geometry>
+      <material name="blue"/>
     </visual>
     <!-- back_caster_collision -->
@@ -55,4 +58,5 @@
         <sphere radius="0.05"/>
       </geometry>
+      <material name="red"/>
     </visual>
     <!-- front_caster_collision -->
@@ -78,4 +82,5 @@
         <sphere radius="0.05"/>
       </geometry>
+      <material name="red"/>
     </visual>
   </link>
@@ -112,4 +117,5 @@
         <cylinder radius="0.1" length="0.05"/>
       </geometry>
+      <material name="black"/>
     </visual>
   </link>
@@ -154,4 +160,5 @@
         <cylinder radius="0.1" length="0.05"/>
       </geometry>
+      <material name="black"/>
     </visual>
   </link>
@@ -186,4 +193,5 @@
         <box size="0.05 0.05 0.05"/>
       </geometry>
+      <material name="blue"/>
     </visual>
   </link>

Commit message: prgs: arranged URDF

File: src/udacity_bot/urdf/udacity_bot.xacro (robot description, xacro)
@@ -2,6 +2,7 @@
 <!-- Udacity Robot -->
 <robot name="udacity_bot" xmlns:xacro="http://www.ros.org/wiki/xacro">
-  <!-- material properties -->
+  <!-- import URDF files -->
   <xacro:include filename="$(find udacity_bot)/urdf/common_properties.xacro"/>
+  <xacro:include filename="$(find udacity_bot)/urdf/udacity_bot.gazebo" />
   <!-- robot_footprint -->
   <link name="robot_footprint"></link>
@@ -14,4 +15,10 @@
   <link name='chassis'>
     <pose>0 0 0.1 0 0 0</pose>
+    <visual name='chassis_visual'>
+      <origin xyz="0 0 0" rpy=" 0 0 0"/>
+      <geometry>
+        <box size=".4 .2 .1"/>
+      </geometry>
+    </visual>
     <inertial>
       <mass value="15.0"/>
@@ -29,12 +36,11 @@
       </geometry>
     </collision>
-    <visual name='chassis_visual'>
-      <origin xyz="0 0 0" rpy=" 0 0 0"/>
-      <geometry>
-        <box size=".4 .2 .1"/>
-      </geometry>
-      <material name="blue"/>
-    </visual>
     <!-- back_caster_collision -->
+    <visual name='back_caster_visual'>
+      <origin xyz="-0.15 0 -0.05" rpy=" 0 0 0"/>
+      <geometry>
+        <sphere radius="0.05"/>
+      </geometry>
+    </visual>
     <collision name='back_caster_collision'>
       <origin xyz="-0.15 0 -0.05" rpy=" 0 0 0"/>
@@ -53,12 +59,11 @@
       </surface>
     </collision>
-    <visual name='back_caster_visual'>
-      <origin xyz="-0.15 0 -0.05" rpy=" 0 0 0"/>
-      <geometry>
-        <sphere radius="0.05"/>
-      </geometry>
-      <material name="red"/>
-    </visual>
     <!-- front_caster_collision -->
+    <visual name='front_caster_visual'>
+      <origin xyz="0.15 0 -0.05" rpy=" 0 0 0"/>
+      <geometry>
+        <sphere radius="0.05"/>
+      </geometry>
+    </visual>
     <collision name='front_caster_collision'>
       <origin xyz="0.15 0 -0.05" rpy=" 0 0 0"/>
@@ -77,11 +82,4 @@
       </surface>
     </collision>
-    <visual name='front_caster_visual'>
-      <origin xyz="0.15 0 -0.05" rpy=" 0 0 0"/>
-      <geometry>
-        <sphere radius="0.05"/>
-      </geometry>
-      <material name="red"/>
-    </visual>
   </link>
   <!-- left_wheel -->
@@ -117,5 +115,4 @@
         <cylinder radius="0.1" length="0.05"/>
       </geometry>
-      <material name="black"/>
     </visual>
   </link>
@@ -160,5 +157,4 @@
         <cylinder radius="0.1" length="0.05"/>
       </geometry>
-      <material name="black"/>
     </visual>
   </link>
@@ -193,5 +189,4 @@
         <box size="0.05 0.05 0.05"/>
       </geometry>
-      <material name="blue"/>
     </visual>
   </link>

Commit message: prgs: issue of material

File: src/udacity_bot/urdf/udacity_bot.xacro (robot description, xacro)
@@ -3,5 +3,5 @@
 <robot name="udacity_bot" xmlns:xacro="http://www.ros.org/wiki/xacro">
   <!-- import URDF files -->
-  <xacro:include filename="$(find udacity_bot)/urdf/common_properties.xacro"/>
+  <!--<xacro:include filename="$(find udacity_bot)/urdf/common_properties.xacro"/>-->
   <xacro:include filename="$(find udacity_bot)/urdf/udacity_bot.gazebo" />
   <!-- robot_footprint -->
@@ -85,4 +85,10 @@
   <!-- left_wheel -->
   <link name="left_wheel">
+    <visual name='left_wheel_visual'>
+      <origin xyz="0 0 0" rpy=" 0 1.5707 1.5707"/>
+      <geometry>
+        <cylinder radius="0.1" length="0.05"/>
+      </geometry>
+    </visual>
    <collision name='left_wheel_collision'>
       <origin xyz="0 0 0" rpy=" 0 1.5707 1.5707"/>
@@ -90,15 +96,5 @@
         <cylinder radius="0.1" length="0.05"/>
       </geometry>
-      <surface>
-        <friction>
-          <ode>
-            <mu>0</mu>
-            <mu2>0</mu2>
-            <slip1>1.0</slip1>
-            <slip2>1.0</slip2>
-          </ode>
-        </friction>
-      </surface>
-    </collision>
+   </collision>
     <inertial>
       <mass value="5.0"/>
@@ -110,10 +106,4 @@
       />
     </inertial>
-    <visual name='left_wheel_visual'>
-      <origin xyz="0 0 0" rpy=" 0 1.5707 1.5707"/>
-      <geometry>
-        <cylinder radius="0.1" length="0.05"/>
-      </geometry>
-    </visual>
   </link>
   <joint type="continuous" name="left_wheel_hinge">
@@ -127,4 +117,10 @@
   <!-- right_wheel -->
   <link name="right_wheel">
+    <visual name='right_wheel_visual'>
+      <origin xyz="0 0 0" rpy=" 0 1.5707 1.5707"/>
+      <geometry>
+        <cylinder radius="0.1" length="0.05"/>
+      </geometry>
+    </visual>
    <collision name='right_wheel_collision'>
       <origin xyz="0 0 0" rpy=" 0 1.5707 1.5707"/>
@@ -132,14 +128,4 @@
         <cylinder radius="0.1" length="0.05"/>
       </geometry>
-      <surface>
-        <friction>
-          <ode>
-            <mu>0</mu>
-            <mu2>0</mu2>
-            <slip1>1.0</slip1>
-            <slip2>1.0</slip2>
-          </ode>
-        </friction>
-      </surface>
     </collision>
     <inertial>
@@ -152,10 +138,4 @@
       />
     </inertial>
-    <visual name='right_wheel_visual'>
-      <origin xyz="0 0 0" rpy=" 0 1.5707 1.5707"/>
-      <geometry>
-        <cylinder radius="0.1" length="0.05"/>
-      </geometry>
-    </visual>
   </link>
   <joint type="continuous" name="right_wheel_hinge">
@@ -169,4 +149,10 @@
   <!-- camera -->
   <link name="camera">
+    <visual name='camera_visual'>
+      <origin xyz="0 0 0" rpy=" 0 0 0"/>
+      <geometry>
+        <box size="0.05 0.05 0.05"/>
+      </geometry>
+    </visual>
    <collision name='camera_collision'>
       <origin xyz="0 0 0" rpy=" 0 0 0"/>
@@ -184,10 +170,4 @@
       />
     </inertial>
-    <visual name='camera_visual'>
-      <origin xyz="0 0 0" rpy=" 0 0 0"/>
-      <geometry>
-        <box size="0.05 0.05 0.05"/>
-      </geometry>
-    </visual>
   </link>
   <joint type="fixed" name="camera_joint">
@@ -199,4 +179,10 @@
   <!-- hokuyo laser range finder -->
   <link name="hokuyo">
+    <visual name='hokuyo_visual'>
+      <origin xyz="0 0 0" rpy=" 0 0 0"/>
+      <geometry>
+        <mesh filename="package://udacity_bot/meshes/hokuyo.dae"/>
+      </geometry>
+    </visual>
     <collision name='hokuyo_collision'>
       <origin xyz="0 0 0" rpy=" 0 0 0"/>
@@ -214,10 +200,4 @@
       />
     </inertial>
-    <visual name='hokuyo_visual'>
-      <origin xyz="0 0 0" rpy=" 0 0 0"/>
-      <geometry>
-        <mesh filename="package://udacity_bot/meshes/hokuyo.dae"/>
-      </geometry>
-    </visual>
   </link>
   <joint type="fixed" name="hokuyo_joint">

Commit message: progs: material issue

File: src/udacity_bot/urdf/udacity_bot.xacro (robot description, xacro)
@@ -90,4 +90,5 @@
         <cylinder radius="0.1" length="0.05"/>
       </geometry>
+      <material name="blue"/>
     </visual>
    <collision name='left_wheel_collision'>

Commit message: progs: done gazebo plugin

File: src/udacity_bot/urdf/udacity_bot.xacro (robot description, xacro)
@@ -124,5 +124,5 @@
       </geometry>
     </visual>
-   <collision name='right_wheel_collision'>
+    <collision name='right_wheel_collision'>
       <origin xyz="0 0 0" rpy=" 0 1.5707 1.5707"/>
       <geometry>

Commit message: progs: added rviz

File: src/udacity_bot/urdf/udacity_bot.xacro (robot description, xacro)
@@ -123,4 +123,5 @@
         <cylinder radius="0.1" length="0.05"/>
       </geometry>
+      <material name="blue"/>
     </visual>
     <collision name='right_wheel_collision'>

Commit message: progs: added AMCL config

File: src/udacity_bot/urdf/udacity_bot.xacro (robot description, xacro)
@@ -160,5 +160,5 @@
       <origin xyz="0 0 0" rpy=" 0 0 0"/>
       <geometry>
-        <box size="0.05"/>
+        <box size="0.05 0.05 0.05"/>
       </geometry>
     </collision>

Commit message: progs: adjusted cater rad

File: src/udacity_bot/urdf/udacity_bot.xacro (robot description, xacro)
@@ -46,5 +46,5 @@
       <origin xyz="-0.15 0 -0.05" rpy=" 0 0 0"/>
       <geometry>
-        <sphere radius="0.05"/>
+        <sphere radius="0.0499"/>
       </geometry>
       <surface>
@@ -69,5 +69,5 @@
       <origin xyz="0.15 0 -0.05" rpy=" 0 0 0"/>
       <geometry>
-        <sphere radius="0.05"/>
+        <sphere radius="0.0499"/>
       </geometry>
       <surface>
