Commit message: progs: fixed material issue

File: src/udacity_bot/urdf/common_properties.xacro (robot description, xacro)
@@ -1,35 +1,15 @@
 <?xml version="1.0" ?>
-<robot name="xacro_properties" xmlns:xacro="http://ros.org/wiki/xacro">
-  <xacro:property name="M_PI" value="3.1415926535897931" />
-  <!-- Init colour -->
+<robot name="udacity_bot" xmlns:xacro="http://www.ros.org/wiki/xacro">
   <material name="black">
       <color rgba="0.0 0.0 0.0 1.0"/>
   </material>
-  <material name="dark">
-    <color rgba="0.3 0.3 0.3 1.0"/>
-  </material>
-  <material name="light_black">
-    <color rgba="0.4 0.4 0.4 1.0"/>
-  </material>
   <material name="blue">
-    <color rgba="0.0 0.0 0.8 1.0"/>
+    <color rgba="0.0 0.0 1.0 1.0"/>
   </material>
   <material name="green">
-    <color rgba="0.0 0.8 0.0 1.0"/>
-  </material>
-  <material name="grey">
-    <color rgba="0.5 0.5 0.5 1.0"/>
-  </material>
-  <material name="orange">
-    <color rgba="${255/255} ${108/255} ${10/255} 1.0"/>
-  </material>
-  <material name="brown">
-    <color rgba="${222/255} ${207/255} ${195/255} 1.0"/>
+    <color rgba="0.0 1.0 0.0 1.0"/>
   </material>
   <material name="red">
-    <color rgba="0.8 0.0 0.0 1.0"/>
-  </material>
-  <material name="white">
-    <color rgba="1.0 1.0 1.0 1.0"/>
+    <color rgba="1.0 0.0 0.0 1.0"/>
   </material>
 </robot>

File: src/udacity_bot/urdf/udacity_bot.xacro (robot description, xacro)
@@ -3,5 +3,5 @@
 <robot name="udacity_bot" xmlns:xacro="http://www.ros.org/wiki/xacro">
   <!-- import URDF files -->
-  <!--<xacro:include filename="$(find udacity_bot)/urdf/common_properties.xacro"/>-->
+  <xacro:include filename="$(find udacity_bot)/urdf/common_properties.xacro"/>
   <xacro:include filename="$(find udacity_bot)/urdf/udacity_bot.gazebo" />
   <!-- robot_footprint -->
@@ -20,4 +20,5 @@
         <box size=".4 .2 .1"/>
       </geometry>
+      <material name="green"/>
     </visual>
     <inertial>
@@ -90,5 +91,5 @@
         <cylinder radius="0.1" length="0.05"/>
       </geometry>
-      <material name="blue"/>
+      <material name="black"/>
     </visual>
    <collision name='left_wheel_collision'>
@@ -123,5 +124,5 @@
         <cylinder radius="0.1" length="0.05"/>
       </geometry>
-      <material name="blue"/>
+      <material name="black"/>
     </visual>
     <collision name='right_wheel_collision'>
