Commit message: progs: muth_bot updated

File: src/muth_bot/urdf/muth_bot.xacro (robot description, xacro)
@@ -31,5 +31,5 @@
       />
     </inertial>
-    <collision name='collision'>
+    <collision name='chassis_collision'>
       <origin xyz="0 0 0" rpy=" 0 0 0"/>
       <geometry>
@@ -37,61 +37,15 @@
       </geometry>
     </collision>
-    <!-- back_caster_collision -->
-    <visual name='back_caster_visual'>
-      <origin xyz="-0.15 0 -0.05" rpy=" 0 0 0"/>
-      <geometry>
-        <sphere radius="0.05"/>
-      </geometry>
-    </visual>
-    <collision name='back_caster_collision'>
-      <origin xyz="-0.15 0 -0.05" rpy=" 0 0 0"/>
-      <geometry>
-        <sphere radius="0.0499"/>
-      </geometry>
-      <surface>
-        <friction>
-          <ode>
-            <mu>0</mu>
-            <mu2>0</mu2>
-            <slip1>1.0</slip1>
-            <slip2>1.0</slip2>
-          </ode>
-        </friction>
-      </surface>
-    </collision>
-    <!-- front_caster_collision -->
-    <visual name='front_caster_visual'>
-      <origin xyz="0.15 0 -0.05" rpy=" 0 0 0"/>
-      <geometry>
-        <sphere radius="0.05"/>
-      </geometry>
-    </visual>
-    <collision name='front_caster_collision'>
-      <origin xyz="0.15 0 -0.05" rpy=" 0 0 0"/>
-      <geometry>
-        <sphere radius="0.0499"/>
-      </geometry>
-      <surface>
-        <friction>
-          <ode>
-            <mu>0</mu>
-            <mu2>0</mu2>
-            <slip1>1.0</slip1>
-            <slip2>1.0</slip2>
-          </ode>
-        </friction>
-      </surface>
-    </collision>
-  </link>
-  <!-- left_wheel -->
-  <link name="left_wheel">
-    <visual name='left_wheel_visual'>
-      <origin xyz="0 0 0" rpy=" 0 1.5707 1.5707"/>
-      <geometry>
-        <cylinder radius="0.1" length="0.05"/>
-      </geometry>
-      <material name="black"/>
-    </visual>
-   <collision name='left_wheel_collision'>
+  </link>
+  <!-- front_left_wheel -->
+  <link name="front_left_wheel">
+    <visual name='front_left_wheel_visual'>
+      <origin xyz="0 0 0" rpy=" 0 1.5707 1.5707"/>
+      <geometry>
+        <cylinder radius="0.1" length="0.05"/>
+      </geometry>
+      <material name="black"/>
+    </visual>
+   <collision name='front_left_wheel_collision'>
       <origin xyz="0 0 0" rpy=" 0 1.5707 1.5707"/>
       <geometry>
@@ -109,40 +63,106 @@
     </inertial>
   </link>
-  <joint type="continuous" name="left_wheel_hinge">
-      <origin xyz="0 0.15 0" rpy="0 0 0"/>
-      <child link="left_wheel"/>
-      <parent link="chassis"/>
-      <axis xyz="0 1 0" rpy="0 0 0"/>
-      <limit effort="10000" velocity="1000"/>
-      <joint_properties damping="1.0" friction="1.0"/>
-  </joint>
-  <!-- right_wheel -->
-  <link name="right_wheel">
-    <visual name='right_wheel_visual'>
-      <origin xyz="0 0 0" rpy=" 0 1.5707 1.5707"/>
-      <geometry>
-        <cylinder radius="0.1" length="0.05"/>
-      </geometry>
-      <material name="black"/>
-    </visual>
-    <collision name='right_wheel_collision'>
-      <origin xyz="0 0 0" rpy=" 0 1.5707 1.5707"/>
-      <geometry>
-        <cylinder radius="0.1" length="0.05"/>
-      </geometry>
-    </collision>
-    <inertial>
-      <mass value="5.0"/>
-      <origin xyz="0.0 0 0" rpy=" 0 1.5707 1.5707"/>
-      <inertia
-          ixx="0.1" ixy="0" ixz="0"
-          iyy="0.1" iyz="0"
-          izz="0.1"
-      />
-    </inertial>
-  </link>
-  <joint type="continuous" name="right_wheel_hinge">
-      <origin xyz="0 -0.15 0" rpy="0 0 0"/>
-      <child link="right_wheel"/>
+  <joint type="continuous" name="front_left_wheel_joint">
+      <origin xyz="0.15 0.15 0" rpy="0 0 0"/>
+      <child link="front_left_wheel"/>
+      <parent link="chassis"/>
+      <axis xyz="0 1 0" rpy="0 0 0"/>
+      <limit effort="10000" velocity="1000"/>
+      <joint_properties damping="1.0" friction="1.0"/>
+  </joint>
+  <!-- front_right_wheel -->
+  <link name="front_right_wheel">
+    <visual name='front_right_wheel_visual'>
+      <origin xyz="0 0 0" rpy=" 0 1.5707 1.5707"/>
+      <geometry>
+        <cylinder radius="0.1" length="0.05"/>
+      </geometry>
+      <material name="black"/>
+    </visual>
+    <collision name='front_right_wheel_collision'>
+      <origin xyz="0 0 0" rpy=" 0 1.5707 1.5707"/>
+      <geometry>
+        <cylinder radius="0.1" length="0.05"/>
+      </geometry>
+    </collision>
+    <inertial>
+      <mass value="5.0"/>
+      <origin xyz="0.0 0 0" rpy=" 0 1.5707 1.5707"/>
+      <inertia
+          ixx="0.1" ixy="0" ixz="0"
+          iyy="0.1" iyz="0"
+          izz="0.1"
+      />
+    </inertial>
+  </link>
+  <joint type="continuous" name="front_right_wheel_joint">
+      <origin xyz="0.15 -0.15 0" rpy="0 0 0"/>
+      <child link="front_right_wheel"/>
+      <parent link="chassis"/>
+      <axis xyz="0 1 0" rpy="0 0 0"/>
+      <limit effort="10000" velocity="1000"/>
+      <joint_properties damping="1.0" friction="1.0"/>
+  </joint>
+  <!-- back_left_wheel -->
+  <link name="back_left_wheel">
+    <visual name='back_left_wheel_visual'>
+      <origin xyz="0 0 0" rpy=" 0 1.5707 1.5707"/>
+      <geometry>
+        <cylinder radius="0.1" length="0.05"/>
+      </geometry>
+      <material name="black"/>
+    </visual>
+   <collision name='back_left_wheel_collision'>
+      <origin xyz="0 0 0" rpy=" 0 1.5707 1.5707"/>
+      <geometry>
+        <cylinder radius="0.1" length="0.05"/>
+      </geometry>
+   </collision>
+    <inertial>
+      <mass value="5.0"/>
+      <origin xyz="0.0 0 0" rpy=" 0 1.5707 1.5707"/>
+      <inertia
+          ixx="0.1" ixy="0" ixz="0"
+          iyy="0.1" iyz="0"
+          izz="0.1"
+      />
+    </inertial>
+  </link>
+  <joint type="continuous" name="back_left_wheel_joint">
+      <origin xyz="-0.15 0.15 0" rpy="0 0 0"/>
+      <child link="back_left_wheel"/>
+      <parent link="chassis"/>
+      <axis xyz="0 1 0" rpy="0 0 0"/>
+      <limit effort="10000" velocity="1000"/>
+      <joint_properties damping="1.0" friction="1.0"/>
+  </joint>
+  <!-- back_right_wheel -->
+  <link name="back_right_wheel">
+    <visual name='back_right_wheel_visual'>
+      <origin xyz="0 0 0" rpy=" 0 1.5707 1.5707"/>
+      <geometry>
+        <cylinder radius="0.1" length="0.05"/>
+      </geometry>
+      <material name="black"/>
+    </visual>
+    <collision name='back_right_wheel_collision'>
+      <origin xyz="0 0 0" rpy=" 0 1.5707 1.5707"/>
+      <geometry>
+        <cylinder radius="0.1" length="0.05"/>
+      </geometry>
+    </collision>
+    <inertial>
+      <mass value="5.0"/>
+      <origin xyz="0.0 0 0" rpy=" 0 1.5707 1.5707"/>
+      <inertia
+          ixx="0.1" ixy="0" ixz="0"
+          iyy="0.1" iyz="0"
+          izz="0.1"
+      />
+    </inertial>
+  </link>
+  <joint type="continuous" name="back_right_wheel_joint">
+      <origin xyz="-0.15 -0.15 0" rpy="0 0 0"/>
+      <child link="back_right_wheel"/>
       <parent link="chassis"/>
       <axis xyz="0 1 0" rpy="0 0 0"/>
@@ -205,5 +225,5 @@
   </link>
   <joint type="fixed" name="hokuyo_joint">
-      <origin xyz="0.15 0 0.1" rpy="0 0 0"/>
+      <origin xyz="0.15 0 0.15" rpy="0 0 0"/>
       <child link="hokuyo"/>
       <parent link="chassis"/>

Commit message: progs: updated muth_bot model

File: src/muth_bot/urdf/muth_bot.xacro (robot description, xacro)
@@ -16,7 +16,7 @@
     <pose>0 0 0.1 0 0 0</pose>
     <visual name='chassis_visual'>
-      <origin xyz="0 0 0" rpy=" 0 0 0"/>
-      <geometry>
-        <box size=".4 .2 .1"/>
+      <origin xyz="0 0 0.05" rpy=" 0 0 0"/>
+      <geometry>
+        <box size=".4 .2 .15"/>
       </geometry>
       <material name="green"/>
@@ -32,7 +32,7 @@
     </inertial>
     <collision name='chassis_collision'>
-      <origin xyz="0 0 0" rpy=" 0 0 0"/>
-      <geometry>
-        <box size=".4 .2 .1"/>
+      <origin xyz="0 0 0.05" rpy=" 0 0 0"/>
+      <geometry>
+        <box size=".4 .2 .15"/>
       </geometry>
     </collision>
@@ -173,5 +173,5 @@
   <link name="camera">
     <visual name='camera_visual'>
-      <origin xyz="0 0 0" rpy=" 0 0 0"/>
+      <origin xyz="0 0 0.05" rpy=" 0 0 0"/>
       <geometry>
         <box size="0.05 0.05 0.05"/>
